File: Editor_Pad.kicad_pcb (KiCad board)
At the start: 2 copper layers, 37 parts, among them SW1 SW_Push, SW10 SW_Push, SW11 SW_Push, SW12 SW_Push, SW13 SW_Push, SW14 SW_Push, SW15 SW_Push, SW16 SW_Push, SW2 SW_Push, SW3 SW_Push, SW4 SW_Push, SW5 SW_Push, SW6 SW_Push, SW7 SW_Push, SW8 SW_Push, SW9 SW_Push

Commit message: Working on a proper routing
Parts:
- added D17: D, Diode_SMD:D_0603_1608Metric_Pad1.05x0.95mm_HandSolder, B.Cu at (135.3, 124.1)
- added D18: D, Diode_SMD:D_0603_1608Metric_Pad1.05x0.95mm_HandSolder, F.Cu at (322.0, 45.5)
- added D19: D, Diode_SMD:D_0603_1608Metric_Pad1.05x0.95mm_HandSolder, B.Cu at (155.6, 51.2)
- added D20: D, Diode_SMD:D_0603_1608Metric_Pad1.05x0.95mm_HandSolder, B.Cu at (155.6, 72.0)
- added D21: D, Diode_SMD:D_0603_1608Metric_Pad1.05x0.95mm_HandSolder, B.Cu at (155.6, 92.3)
- added D22: D, Diode_SMD:D_0603_1608Metric_Pad1.05x0.95mm_HandSolder, B.Cu at (155.6, 112.6)
- added D23: D, Diode_SMD:D_0603_1608Metric_Pad1.05x0.95mm_HandSolder, B.Cu at (177.2, 123.6)
- added D24: D, Diode_SMD:D_0603_1608Metric_Pad1.05x0.95mm_HandSolder, F.Cu at (322.0, 48.0)
- added D25: D, Diode_SMD:D_0603_1608Metric_Pad1.05x0.95mm_HandSolder, B.Cu at (176.8, 42.8)
- added D26: D, Diode_SMD:D_0603_1608Metric_Pad1.05x0.95mm_HandSolder, B.Cu at (176.8, 63.1)
- added D27: D, Diode_SMD:D_0603_1608Metric_Pad1.05x0.95mm_HandSolder, B.Cu at (176.8, 83.2)
- added D28: D, Diode_SMD:D_0603_1608Metric_Pad1.05x0.95mm_HandSolder, B.Cu at (176.8, 103.7)
- added D29: D, Diode_SMD:D_0603_1608Metric_Pad1.05x0.95mm_HandSolder, B.Cu at (211.5, 122.8)
- added D30: D, Diode_SMD:D_0603_1608Metric_Pad1.05x0.95mm_HandSolder, F.Cu at (322.0, 50.6)
- added D31: D, Diode_SMD:D_0603_1608Metric_Pad1.05x0.95mm_HandSolder, F.Cu at (322.0, 53.2)
- added D32: D, Diode_SMD:D_0603_1608Metric_Pad1.05x0.95mm_HandSolder, F.Cu at (322.0, 55.8)
- added D33: D, Diode_SMD:D_0603_1608Metric_Pad1.05x0.95mm_HandSolder, F.Cu at (322.0, 58.4)
- added R5: 10k, Resistor_SMD:R_0603_1608Metric, F.Cu at (243.2, 74.5)
- added R6: 10k, Resistor_SMD:R_0603_1608Metric, F.Cu at (321.8, 61.0)
- added REF**: MountingHole_3.2mm_M3_ISO7380, MountingHole:MountingHole_3.2mm_M3_ISO7380, F.Cu at (40.6, 34.3)
- added REF**: MountingHole_3.2mm_M3_ISO7380, MountingHole:MountingHole_3.2mm_M3_ISO7380, F.Cu at (243.8, 143.5)
- added REF**: MountingHole_3.2mm_M3_ISO7380, MountingHole:MountingHole_3.2mm_M3_ISO7380, F.Cu at (158.8, 34.3)
- added REF**: MountingHole_3.2mm_M3_ISO7380, MountingHole:MountingHole_3.2mm_M3_ISO7380, F.Cu at (118.1, 143.5)
- added SW17: SW_Push, PCM_Switch_Keyboard_Cherry_MX:SW_Cherry_MX_PCB_1.00u, F.Cu at (137.8, 119.4)
- added SW18: SW_Push, Button_Switch_THT:SW_PUSH_6mm, F.Cu at (210.1, 62.2)
- added SW19: SW_Push, PCM_Switch_Keyboard_Cherry_MX:SW_Cherry_MX_PCB_1.00u, F.Cu at (158.4, 47.0)
- added SW20: SW_Push, PCM_Switch_Keyboard_Cherry_MX:SW_Cherry_MX_PCB_1.00u, F.Cu at (158.4, 67.3)
- added SW21: SW_Push, PCM_Switch_Keyboard_Cherry_MX:SW_Cherry_MX_PCB_1.00u, F.Cu at (158.4, 87.6)
- added SW22: SW_Push, PCM_Switch_Keyboard_Cherry_MX:SW_Cherry_MX_PCB_1.00u, F.Cu at (158.4, 108.0)
- added SW23: SW_Push, PCM_Switch_Keyboard_Cherry_MX:SW_Cherry_MX_PCB_1.00u, F.Cu at (179.7, 119.4)
- added SW24: SW_Push, Button_Switch_THT:SW_PUSH_6mm, F.Cu at (210.1, 72.4)
- added SW25: SW_Push, PCM_Switch_Keyboard_Cherry_MX:SW_Cherry_MX_PCB_1.00u, F.Cu at (179.7, 38.1)
- added SW26: SW_Push, PCM_Switch_Keyboard_Cherry_MX:SW_Cherry_MX_PCB_1.00u, F.Cu at (179.7, 58.4)
- added SW27: SW_Push, PCM_Switch_Keyboard_Cherry_MX:SW_Cherry_MX_PCB_1.00u, F.Cu at (179.7, 78.7)
- added SW28: SW_Push, PCM_Switch_Keyboard_Cherry_MX:SW_Cherry_MX_PCB_1.00u, F.Cu at (179.7, 99.0)
- added SW29: SW_Push, PCM_Switch_Keyboard_Cherry_MX:SW_Cherry_MX_PCB_1.00u, F.Cu at (215.3, 139.7)
- added SW30: SW_Push, Button_Switch_THT:SW_PUSH_6mm, F.Cu at (218.4, 41.9)
- added SW31: SW_Push, Button_Switch_THT:SW_PUSH_6mm, F.Cu at (218.4, 52.2)
- added SW32: SW_Push, Button_Switch_THT:SW_PUSH_6mm, F.Cu at (218.4, 62.4)
- added SW33: SW_Push, Button_Switch_THT:SW_PUSH_6mm, F.Cu at (218.4, 72.4)
- A1: value Arduino_Nano_Every_Socket -> Arduino_Uno_R3_Shield; footprint PCM_arduino-library:Arduino_Nano_Every_Socket -> PCM_arduino-library:Arduino_Uno_R3_Shield
- D12, D6, R1, R2, R3, R4: moved to F.Cu
- SW12, SW6: footprint PCM_Switch_Keyboard_Cherry_MX:SW_Cherry_MX_PCB_1.00u -> Button_Switch_THT:SW_PUSH_6mm
- moved D12 261.7 mm to (322.0, 42.9), turned to 0 degrees
- moved D6 210.3 mm to (322.0, 40.3), turned to 0 degrees
- moved SW12 179.5 mm to (210.1, 52.1), turned to 90 degrees
- moved D4 125.1 mm to (42.5, 121.9), turned to 90 degrees
- moved SW6 117.8 mm to (210.1, 41.9), turned to 90 degrees
- moved SW11 109.9 mm to (71.8, 139.7)
- moved SW4 109.3 mm to (46.4, 118.1)
- moved SW15 107.8 mm to (137.8, 78.7)
- moved D14 101.0 mm to (134.9, 63.1), turned to 90 degrees
- moved D13 98.4 mm to (134.9, 42.3), turned to 90 degrees
- moved SW16 96.2 mm to (137.8, 99.0)
- moved D15 92.7 mm to (134.9, 83.4), turned to 90 degrees
- moved SW14 91.6 mm to (137.8, 58.4)
- moved SW13 90.4 mm to (137.8, 38.1)
- moved D16 83.3 mm to (134.9, 103.7), turned to 90 degrees
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Connections:
- A1 pad D10: ROW 1 -> COL 4
- A1 pad D11: ROW 2 -> COL 3
- A1 pad D12: ROW 3 -> COL 2
- A1 pad D13: ROW 4 -> COL 1
- A1 pad D2: COL 1 -> ROW 6
- A1 pad D3: COL 2 -> ROW 5
- A1 pad D4: COL 3 -> ROW 4
- A1 pad D5: COL 4 -> ROW 3
- A1 pad D6: unconnected-(A1-PadD6) -> ROW 2
- A1 pad D7: unconnected-(A1-PadD7) -> ROW 1
- A1 pad D8: unconnected-(A1-PadD8) -> COL 6
- A1 pad D9: unconnected-(A1-PadD9) -> COL 5
- D11 pad 1: ROW 3 -> ROW 5
- D12 pad 1: ROW 4 -> ROW 6
- D13 pad 1: ROW 3 -> ROW 1
- D14 pad 1: ROW 4 -> ROW 2
- D2 pad 1: ROW 1 -> ROW 2
- D3 pad 1: ROW 1 -> ROW 3
- D4 pad 1: ROW 1 -> ROW 4
- D5 pad 1: ROW 2 -> ROW 5
- D6 pad 1: ROW 2 -> ROW 6
- D7 pad 1: ROW 2 -> ROW 1
- SW10 pad 1: Net-(D11-A) -> Net-(D10-A)
- SW11 pad 1: Net-(D13-A) -> Net-(D11-A)
- SW11 pad 2: COL 3 -> COL 2
- SW12 pad 1: Net-(D15-A) -> Net-(D12-A)
- SW12 pad 2: COL 4 -> COL 2
- SW13 pad 1: Net-(D10-A) -> Net-(D13-A)
- SW13 pad 2: COL 1 -> COL 3
- SW14 pad 1: Net-(D12-A) -> Net-(D14-A)
- SW14 pad 2: COL 2 -> COL 3
- SW15 pad 1: Net-(D14-A) -> Net-(D15-A)
- SW16 pad 2: COL 4 -> COL 3
- SW2 pad 2: COL 2 -> COL 1
- SW3 pad 2: COL 3 -> COL 1
- SW4 pad 2: COL 4 -> COL 1
- SW6 pad 2: COL 2 -> COL 1
- SW7 pad 2: COL 3 -> COL 2
- SW8 pad 2: COL 4 -> COL 2
- SW9 pad 2: COL 1 -> COL 2
Routing:
- net ROW 5: track 0.00 -> 238.5 mm
- net COL 5: track 0.00 -> 219.9 mm
- net ROW 3: track 19.2 -> 195.2 mm
- net ROW 2: track 84.2 -> 207.4 mm
- net ROW 1: track 112.0 -> 228.9 mm
- net COL 1: track 212.8 -> 320.5 mm
- net COL 4: track 297.4 -> 214.0 mm
- net COL 2: track 237.0 -> 314.1 mm
- net ROW 4: track 195.4 -> 251.3 mm
- net +5V: track 19.3 -> 69.0 mm, vias 1 -> 6
- net COL 3: track 240.7 -> 224.4 mm
- net Net-(D29-A): track 0.00 -> 14.0 mm
- net Net-(D6-A): track 13.7 -> 0.00 mm
- net Net-(D12-A): track 11.4 -> 0.00 mm
- net Net-(D8-A): track 14.3 -> 5.44 mm
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Other:
- board outline added: 217.2 x 124.5 mm
- board text removed: "inversser les lignes"

Commit message: Slightly modified
Parts:
- removed A1: Arduino_Uno_R3_Shield, PCM_arduino-library:Arduino_Uno_R3_Shield
- removed REF** (x4): MountingHole_3.2mm_M3_ISO7380, MountingHole:MountingHole_3.2mm_M3_ISO7380
- added A2: Arduino_UNO_R3, Module:Arduino_UNO_R3, B.Cu at (179.1, 48.6)
- added M3: MountingHole_3.2mm_M3_DIN965_Pad, MountingHole:MountingHole_3.2mm_M3_DIN965_Pad, F.Cu at (34.3, 25.4)
- added M3: MountingHole_3.2mm_M3_DIN965_Pad, MountingHole:MountingHole_3.2mm_M3_DIN965_Pad, F.Cu at (227.3, 144.1)
- D12, D18, D24, D30, D31, D32, D33, D6: moved to B.Cu
- SW12, SW18, SW24, SW6: footprint Button_Switch_THT:SW_PUSH_6mm -> PCM_Switch_Keyboard_Cherry_MX:SW_Cherry_MX_PCB_1.00u
- SW25, SW26, SW27, SW28: footprint PCM_Switch_Keyboard_Cherry_MX:SW_Cherry_MX_PCB_1.00u -> Button_Switch_THT:SW_PUSH_6mm
- moved D12 294.1 mm to (37.9, 118.7)
- moved D6 284.2 mm to (38.7, 63.9), turned to 90 degrees
- moved D18 277.3 mm to (62.2, 142.5), turned to 90 degrees
- moved D24 253.2 mm to (87.0, 142.5), turned to 90 degrees
- moved SW12 179.8 mm to (41.9, 115.6), turned to 0 degrees
- moved SW6 169.2 mm to (41.9, 59.7), turned to 0 degrees
- moved SW18 163.6 mm to (65.4, 138.4), turned to 0 degrees
- moved SW24 136.9 mm to (90.2, 138.4), turned to 0 degrees
- moved D33 114.4 mm to (208.5, 73.0), turned to 180 degrees
- moved D30 114.3 mm to (208.5, 36.8), turned to 180 degrees
- moved D32 113.6 mm to (208.5, 61.0), turned to 180 degrees
- moved D31 113.5 mm to (208.5, 48.9), turned to 180 degrees
- moved R6 100.1 mm to (221.6, 61.4), turned to -90 degrees
- moved D17 98.3 mm to (38.7, 142.6)
- moved SW17 97.8 mm to (41.9, 138.4)
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Connections:
- D30 pad 1: ROW 6 -> ROW 1
- D31 pad 1: ROW 1 -> ROW 2
- D32 pad 1: ROW 2 -> ROW 3
- D33 pad 1: ROW 3 -> ROW 4
- SW30 pad 2: COL 5 -> COL 6
Routing:
- net ROW 6: track 0.00 -> 332.8 mm
- net COL 3: track 224.4 -> 305.8 mm
- net COL 5: track 219.9 -> 146.0 mm
- net ROW 5: track 238.5 -> 310.0 mm
- net ROW 1: track 228.9 -> 290.3 mm
- net COL 6: track 0.00 -> 58.8 mm, vias 0 -> 1
- net COL 4: track 214.0 -> 267.8 mm
- net ROW 4: track 251.3 -> 201.6 mm
- net +5V: track 69.0 -> 118.1 mm
- net COL 1: track 320.5 -> 289.0 mm
- net COL 2: track 314.1 -> 293.4 mm
- net ROW 3: track 195.2 -> 185.2 mm
- net Net-(D32-A): track 0.00 -> 9.03 mm
- net Net-(D31-A): track 0.00 -> 9.03 mm
- net Net-(D30-A): track 0.00 -> 9.03 mm
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- added copper zone on B.Cu, net GND
- added copper zone on F.Cu, net GND
Other:
- board size 217.2 x 124.5 mm -> 203.2 x 128.9 mm
