File: pb_matrix.kicad_sch (KiCad schematic)
At the start: 36 parts, among them SW1 SW_Push, SW10 SW_Push, SW11 SW_Push, SW12 SW_Push, SW13 SW_Push, SW14 SW_Push, SW15 SW_Push, SW16 SW_Push, SW2 SW_Push, SW3 SW_Push, SW4 SW_Push, SW5 SW_Push, SW6 SW_Push, SW7 SW_Push, SW8 SW_Push, SW9 SW_Push

Commit message: Working on a proper routing
Parts:
- added D11, D12, D17, D18, D23, D24, D25, D26, D27, D28, D29, D30, D31, D32, D33, D5, D6: D, Diode_SMD:D_0603_1608Metric_Pad1.05x0.95mm_HandSolder, symbol Device:D
- added R5, R6: 10k, Resistor_SMD:R_0603_1608Metric, symbol Device:R
- added SW11, SW17, SW23, SW25, SW26, SW27, SW28, SW29, SW5: SW_Push, PCM_Switch_Keyboard_Cherry_MX:SW_Cherry_MX_PCB_1.00u, symbol Switch:SW_Push
- added SW12, SW18, SW24, SW30, SW31, SW32, SW33, SW6: SW_Push, Button_Switch_THT:SW_PUSH_6mm, symbol Switch:SW_Push
- renumbered D12 to D10, D3 to D13, D7 to D14, D13 to D15, D14 to D16, D4 to D19, D5 to D2, D8 to D20, D15 to D21, D16 to D22, D9 to D3, D10 to D4, D2 to D7, D6 to D8, D11 to D9, SW14 to SW10, SW3 to SW13, SW7 to SW14, SW11 to SW15, SW15 to SW16, SW4 to SW19, SW5 to SW2, SW8 to SW20, SW12 to SW21, SW16 to SW22, SW9 to SW3, SW13 to SW4, SW2 to SW7, SW6 to SW8, SW10 to SW9
Connections:
- net +5V: now also R5.1, R6.1
- net COL 1: now also SW5.2, SW6.2
- net COL 2: now also SW11.2, SW12.2
- net COL 3: now also SW17.2, SW18.2
- net COL 4: now also SW23.2, SW24.2
- net ROW 1: now also D25.1 (K), D31.1 (K)
- net ROW 2: now also D26.1 (K), D32.1 (K)
- net ROW 3: now also D27.1 (K), D33.1 (K)
- net ROW 4: now also D28.1 (K)
- new net: D11.2 (A), SW11.1
- new net: D5.2 (A), SW5.1
- new net: D27.2 (A), SW27.1
- new net: D32.2 (A), SW32.1
- new net: D12.2 (A), SW12.1
- new net: D30.2 (A), SW30.1
- new net: D29.2 (A), SW29.1
- new net: D18.2 (A), SW18.1
- new net: D6.2 (A), SW6.1
- new net: D23.2 (A), SW23.1
- new net: D26.2 (A), SW26.1
- new net: D24.2 (A), SW24.1
- new net: D28.2 (A), SW28.1
- new net: D17.2 (A), SW17.1
- new net: D25.2 (A), SW25.1
- new net: D31.2 (A), SW31.1
- new net: D33.2 (A), SW33.1
- new net COL 5: R5.2, SW25.2, SW26.2, SW27.2, SW28.2, SW29.2, SW30.2
- new net COL 6: R6.2, SW31.2, SW32.2, SW33.2
- new net ROW 5: D11.1 (K), D17.1 (K), D23.1 (K), D29.1 (K), D5.1 (K)
- new net ROW 6: D12.1 (K), D18.1 (K), D24.1 (K), D30.1 (K), D6.1 (K)
Other:
- moved on the sheet: D1, D10, D13, D14, D15, D16, D19, D2, D20, D21, D22, D3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

Commit message: Slightly modified
Parts:
- removed SW30, SW6: SW_Push, Button_Switch_THT:SW_PUSH_6mm, symbol Switch:SW_Push
- added SW24, SW29: SW_Push, PCM_Switch_Keyboard_Cherry_MX:SW_Cherry_MX_PCB_1.00u, symbol Switch:SW_Push
- SW25, SW26: footprint PCM_Switch_Keyboard_Cherry_MX:SW_Cherry_MX_PCB_1.00u -> Button_Switch_THT:SW_PUSH_6mm
- renumbered D30 to D24, D31 to D30, D32 to D31, D33 to D32, D24 to D33, SW28 to SW12, SW29 to SW18, SW18 to SW27, SW12 to SW28, SW31 to SW30, SW32 to SW31, SW33 to SW32, SW24 to SW33, SW27 to SW6
Connections:
- net COL 1: now also SW6.2
- net COL 2: now also SW12.2; no longer SW28.2
- net COL 3: now also SW18.2; no longer SW27.2
- net COL 4: now also SW24.2; no longer SW33.2
- net COL 5: now also SW27.2, SW28.2, SW29.2; no longer SW12.2, SW18.2, SW6.2
- net COL 6: now also SW33.2
- net ROW 4: now also D33.1 (K)
- net ROW 6: no longer D33.1 (K)
- net at D27.2 (A): now also SW27.1; no longer SW6.1
- net at D12.2 (A): now also SW12.1; no longer SW28.1
- net at D24.2 (A): now also SW24.1
- net at D29.2 (A): now also SW29.1; no longer SW18.1
- net at D18.2 (A): now also SW18.1; no longer SW27.1
- net at D6.2 (A): now also SW6.1
- net at D28.2 (A): now also SW28.1; no longer SW12.1
Other:
- moved on the sheet: D24, D33, SW12, SW18, SW27, SW28, SW33, SW6
